File: Hardware/USB_Power_Injector_V1.0/USB_Power_Injector_V1.0.kicad_sch (KiCad schematic)
At the start: 10 parts, among them J1 Red Banana Jack, J2 Black Banana Jack, J3 USB_B, J4 USB_A

Commit message: BOM changes
Excluded the mounting holes and N.F. components from BOM generation. BOM generated.
Parts:
- C1, C2, H1, H2, H3, H4: now left out of the parts list
Changed lines of the file:
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@@
   )
   (symbol (lib_id "Device:C") (at 121.92 43.18 0) (unit 1)
-    (in_bom yes) (on_board yes)
+    (in_bom no) (on_board yes)
     (property "Reference" "C2" (id 0) (at 114.3 41.91 0)
       (effects (font (size 1.27 1.27)) (justify left))
@@
   )
   (symbol (lib_id "Mechanical:MountingHole") (at 53.34 124.46 0) (unit 1)
-    (in_bom yes) (on_board yes) (fields_autoplaced)
+    (in_bom no) (on_board yes) (fields_autoplaced)
     (property "Reference" "H4" (id 0) (at 55.88 123.1899 0)
       (effects (font (size 1.27 1.27)) (justify left))
@@
   )
   (symbol (lib_id "Mechanical:MountingHole") (at 53.34 118.11 0) (unit 1)
-    (in_bom yes) (on_board yes) (fields_autoplaced)
+    (in_bom no) (on_board yes) (fields_autoplaced)
     (property "Reference" "H3" (id 0) (at 55.88 116.8399 0)
       (effects (font (size 1.27 1.27)) (justify left))
@@
   )
   (symbol (lib_id "Mechanical:MountingHole") (at 27.94 124.46 0) (unit 1)
-    (in_bom yes) (on_board yes) (fields_autoplaced)
+    (in_bom no) (on_board yes) (fields_autoplaced)
     (property "Reference" "H2" (id 0) (at 30.48 123.1899 0)
       (effects (font (size 1.27 1.27)) (justify left))
@@
   )
   (symbol (lib_id "Mechanical:MountingHole") (at 27.94 118.11 0) (unit 1)
-    (in_bom yes) (on_board yes) (fields_autoplaced)
+    (in_bom no) (on_board yes) (fields_autoplaced)
     (property "Reference" "H1" (id 0) (at 30.48 116.8399 0)
       (effects (font (size 1.27 1.27)) (justify left))
@@
   )
   (symbol (lib_id "Device:C") (at 133.35 43.18 0) (unit 1)
-    (in_bom yes) (on_board yes)
+    (in_bom no) (on_board yes)
     (property "Reference" "C1" (id 0) (at 125.73 41.91 0)
       (effects (font (size 1.27 1.27)) (justify left))
